File: Design/H3AR1.sch (EAGLE design)
At the start: 8 parts, among them P1 HEXABIT__REVERSED_NO_P3, U1 TPS76433DBVT

Commit message: Update the logo
Parts:
- added TRIMBLE-LOGO1: HEXA-LOGO, HEXABITZ_USER_INTERFACE_PARTS:HEXA-LOGO
